File: pcb/rev2/composite_input.sch (KiCad schematic (older format))
At the start: 19 parts, among them IC28 TVP5150AM1PBS, X1 XTAL_12MHZ_TXC_7A-14.31818MAA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

Commit message: axi4/zynq version: wip
Parts:
- C29, C30, C52, C83: symbol CC0603_1UF_50V_10%_X5R -> dsi_shield-rescue:CC0603_1UF_50V_10%_X5R-
- C31, C59: symbol CC0603_22PF_50V_5%_NP0 -> dsi_shield-rescue:CC0603_22PF_50V_5%_NP0-
- C7, C84, C85, C86: symbol CC0603_100NF_100V_10%_X7R -> dsi_shield-rescue:CC0603_100NF_100V_10%_X7R-
- IC28: symbol TVP5150AM1PBS -> dsi_shield-rescue:TVP5150AM1PBS-
- L1, L6: symbol IND0805_MURATA_BLM21PG221SN1D -> dsi_shield-rescue:IND0805_MURATA_BLM21PG221SN1D-
- R19, R32: symbol R0603_33R_1%_0.1W_100PPM -> dsi_shield-rescue:R0603_33R_1%_0.1W_100PPM-
- R33, R34, R48: symbol R0603_3K3_1%_0.1W_100PPM -> dsi_shield-rescue:R0603_3K3_1%_0.1W_100PPM-
- X1: symbol XTAL_12MHZ_TXC_7A-12.000MAAJ-T -> dsi_shield-rescue:XTAL_12MHZ_TXC_7A-12.000MAAJ-T-
Changed lines of the file:
@@
-EESchema Schematic File Version 2
-LIBS:Capacitors Networks THD
-LIBS:Capacitors Networks SMD
-LIBS:Capacitors THD
-LIBS:Capacitors SMD
-LIBS:Miscellaneous
-LIBS:HARWIN
-LIBS:LEMO
-LIBS:WEIDMULLER
-LIBS:FCI
-LIBS:MOLEX
-LIBS:TYCO
-LIBS:ERNI
-LIBS:MENTOR
-LIBS:SAMTEC
-LIBS:STELVIO-KONTEK COMATEL
-LIBS:AMPHENOL
-LIBS:HARTING
-LIBS:3M
-LIBS:Pads
-LIBS:Switches
-LIBS:Relays
-LIBS:Heat-Sinks
-LIBS:Fasteners & Fixings
-LIBS:Batteries
-LIBS:Fuses
-LIBS:Metal Screening Box
-LIBS:Sockets
-LIBS:Regulators
-LIBS:Transistors
-LIBS:Power Supplies
-LIBS:Analog & Interface
-LIBS:Sensors
-LIBS:Logic
-LIBS:Optocouplers
-LIBS:Standard Logic
-LIBS:DC-DC Converters
-LIBS:Operational Amplifiers
-LIBS:Crystals & Oscillators
-LIBS:Diodes
-LIBS:LEDs & Displays
-LIBS:PCB Modules
-LIBS:Bonding
-LIBS:Resistors THD
-LIBS:Potentiometers SMD
-LIBS:Thermistors And Varistors
-LIBS:Potentiometers THD
-LIBS:Resistor Networks THD
-LIBS:Resistors SMD
-LIBS:Resistor Networks SMD
-LIBS:Transformers
-LIBS:Inductors SMD
-LIBS:Inductors THD
-LIBS:Cores
-LIBS:power
-LIBS:conn
-LIBS:dsi_shield
+EESchema Schematic File Version 4
 LIBS:dsi_shield-cache
 EELAYER 26 0
@@
 $EndDescr
 $Comp
-L TVP5150AM1PBS IC28
+L dsi_shield-rescue:TVP5150AM1PBS- IC28
 U 1 1 59904558
 P 5150 2700
@@
 CVBS_IN
 $Comp
-L R0603_33R_1%_0.1W_100PPM R19
+L dsi_shield-rescue:R0603_33R_1%_0.1W_100PPM- R19
 U 1 1 59905E84
 P 1900 1500
@@
 $EndComp
 $Comp
-L R0603_33R_1%_0.1W_100PPM R32
+L dsi_shield-rescue:R0603_33R_1%_0.1W_100PPM- R32
 U 1 1 59906001
 P 2300 1600
@@
 $EndComp
 $Comp
-L CC0603_100NF_100V_10%_X7R C7
+L dsi_shield-rescue:CC0603_100NF_100V_10%_X7R- C7
 U 1 1 59906E21
 P 2450 1500
@@
 NoConn ~ 4950 2900
 $Comp
-L R0603_3K3_1%_0.1W_100PPM R33
+L dsi_shield-rescue:R0603_3K3_1%_0.1W_100PPM- R33
 U 1 1 5990911E
 P 4250 3100
@@
 $EndComp
 $Comp
-L R0603_3K3_1%_0.1W_100PPM R34
+L dsi_shield-rescue:R0603_3K3_1%_0.1W_100PPM- R34
 U 1 1 5990925B
 P 4250 3200
@@
 $EndComp
 $Comp
-L +3V3 #PWR0111
+L dsi_shield-rescue:+3V3- #PWR0111
 U 1 1 59909459
 P 4050 3100
@@
 $EndComp
 $Comp
-L CC0603_22PF_50V_5%_NP0 C31
+L dsi_shield-rescue:CC0603_22PF_50V_5%_NP0- C31
 U 1 1 5990B552
 P 2850 3600
@@
 $EndComp
 $Comp
-L CC0603_22PF_50V_5%_NP0 C59
+L dsi_shield-rescue:CC0603_22PF_50V_5%_NP0- C59
 U 1 1 5990B6BB
 P 3300 3600
@@
 $EndComp
 $Comp
-L XTAL_12MHZ_TXC_7A-12.000MAAJ-T X1
+L dsi_shield-rescue:XTAL_12MHZ_TXC_7A-12.000MAAJ-T- X1
 U 1 1 5991099D
 P 2350 3400
@@
 SDA
 $Comp
-L GNDA #PWR0114
+L dsi_shield-rescue:GNDA- #PWR0114
 U 1 1 599157A5
 P 7050 5400
@@
 $EndComp
 $Comp
-L GND #PWR0115
+L dsi_shield-rescue:GND- #PWR0115
 U 1 1 5991582A
 P 7250 5400
@@
 $EndComp
 $Comp
-L CC0603_1UF_50V_10%_X5R C29
+L dsi_shield-rescue:CC0603_1UF_50V_10%_X5R- C29
 U 1 1 59918073
 P 3500 4850
@@
 $EndComp
 $Comp
-L CC0603_1UF_50V_10%_X5R C30
+L dsi_shield-rescue:CC0603_1UF_50V_10%_X5R- C30
 U 1 1 59918205
 P 3900 4700
@@
 $EndComp
 $Comp
-L CC0603_1UF_50V_10%_X5R C52
+L dsi_shield-rescue:CC0603_1UF_50V_10%_X5R- C52
 U 1 1 599182A5
 P 3950 5150
@@
 $EndComp
 $Comp
-L GNDA #PWR0116
+L dsi_shield-rescue:GNDA- #PWR0116
 U 1 1 5991843E
 P 3500 5300
@@
 $EndComp
 $Comp
-L GNDA #PWR0117
+L dsi_shield-rescue:GNDA- #PWR0117
 U 1 1 599184B2
 P 3950 5300
@@
 $EndComp
 $Comp
-L +3V3 #PWR0118
+L dsi_shield-rescue:+3V3- #PWR0118
 U 1 1 5991B27D
 P 4950 4750
@@
 $EndComp
 $Comp
-L +1V8 #PWR0119
+L dsi_shield-rescue:+1V8- #PWR0119
 U 1 1 5991B442
 P 4950 4850
@@
 $EndComp
 $Comp
-L VDDA #PWR0120
+L dsi_shield-rescue:VDDA- #PWR0120
 U 1 1 5991BFDF
 P 4750 5050
@@
 $EndComp
 $Comp
-L IND0805_MURATA_BLM21PG221SN1D L1
+L dsi_shield-rescue:IND0805_MURATA_BLM21PG221SN1D- L1
 U 1 1 59920F8F
 P 5750 6100
@@
 $EndComp
 $Comp
-L IND0805_MURATA_BLM21PG221SN1D L6
+L dsi_shield-rescue:IND0805_MURATA_BLM21PG221SN1D- L6
 U 1 1 59920FDD
 P 5750 6400
@@
 $EndComp
 $Comp
-L GND #PWR0121
+L dsi_shield-rescue:GND- #PWR0121
 U 1 1 5992109A
 P 5750 6100
@@
 $EndComp
 $Comp
-L GNDA #PWR0122
+L dsi_shield-rescue:GNDA- #PWR0122
 U 1 1 599210CF
 P 6050 6100
@@
 $EndComp
 $Comp
-L +1V8 #PWR0123
+L dsi_shield-rescue:+1V8- #PWR0123
 U 1 1 5992113C
 P 5750 6400
@@
 $EndComp
 $Comp
-L VDDA #PWR0124
+L dsi_shield-rescue:VDDA- #PWR0124
 U 1 1 59921163
 P 6100 6400
@@
 $EndComp
 $Comp
-L CC0603_1UF_50V_10%_X5R C83
+L dsi_shield-rescue:CC0603_1UF_50V_10%_X5R- C83
 U 1 1 5992294C
 P 3450 6200
@@
 $EndComp
 $Comp
-L GNDA #PWR0125
+L dsi_shield-rescue:GNDA- #PWR0125
 U 1 1 599229D3
 P 3450 6600
@@
 $EndComp
 $Comp
-L CC0603_100NF_100V_10%_X7R C84
+L dsi_shield-rescue:CC0603_100NF_100V_10%_X7R- C84
 U 1 1 5992364C
 P 3850 6200
@@
 $EndComp
 $Comp
-L VDDA #PWR0126
+L dsi_shield-rescue:VDDA- #PWR0126
 U 1 1 599239E2
 P 3450 6100
@@
 $EndComp
 $Comp
-L CC0603_100NF_100V_10%_X7R C85
+L dsi_shield-rescue:CC0603_100NF_100V_10%_X7R- C85
 U 1 1 59923A52
 P 4350 6200
@@
 $EndComp
 $Comp
-L CC0603_100NF_100V_10%_X7R C86
+L dsi_shield-rescue:CC0603_100NF_100V_10%_X7R- C86
 U 1 1 59923ADE
 P 4800 6200
@@
 $EndComp
 $Comp
-L GND #PWR0127
+L dsi_shield-rescue:GND- #PWR0127
 U 1 1 59923BEB
 P 4350 6500
@@
 $EndComp
 $Comp
-L GND #PWR0128
+L dsi_shield-rescue:GND- #PWR0128
 U 1 1 59923C98
 P 4800 6500
@@
 $EndComp
 $Comp
-L +1V8 #PWR0129
+L dsi_shield-rescue:+1V8- #PWR0129
 U 1 1 59923E68
 P 4350 6100
@@
 $EndComp
 $Comp
-L +3V3 #PWR0130
+L dsi_shield-rescue:+3V3- #PWR0130
 U 1 1 59924064
 P 4800 6100
@@
 	7700 4000 6950 4000
 $Comp
-L R0603_3K3_1%_0.1W_100PPM R48
+L dsi_shield-rescue:R0603_3K3_1%_0.1W_100PPM- R48
 U 1 1 599279EE
 P 7400 4150
@@
 Connection ~ 7400 4000
 $Comp
-L GND #PWR0131
+L dsi_shield-rescue:GND- #PWR0131
 U 1 1 59927CC9
 P 7400 4450
@@
 Composite input/decoder
 $Comp
-L GNDA #PWR0110
+L dsi_shield-rescue:GNDA- #PWR0110
 U 1 1 599E49EF
 P 2300 2000
@@
 $EndComp
 $Comp
-L GNDA #PWR0112
+L dsi_shield-rescue:GNDA- #PWR0112
 U 1 1 599EEF10
 P 2850 3900
@@
 $EndComp
 $Comp
-L GNDA #PWR0113
+L dsi_shield-rescue:GNDA- #PWR0113
 U 1 1 599EEF41
 P 3300 3900
