File: pcb/rev2/ddr_sdram.sch (KiCad schematic (older format))
At the start: 16 parts, among them IC10 MT46V32M16P-5B:F

Commit message: pcb wip
Parts:
- C11, C65, C67, C71, C72, C73, C75: footprint CAPC1608X90N -> Capacitors SMD:CAPC1608X90N
- C64, C66, C68, C69, C70: footprint CAPC1608X87N -> Capacitors SMD:CAPC1608X87N
- R67, R68, R69: footprint RESC1608X55N -> Resistors SMD:RESC1608X55N
Changed lines of the file:
@@
 F 0 "R67" V 4304 4910 50  0000 L CNN
 F 1 "R0603_100R_1%_0.1W_100PPM" H 4200 4640 60  0001 L CNN
-F 2 "RESC1608X55N" H 4200 3830 60  0001 L CNN
+F 2 "Resistors SMD:RESC1608X55N" H 4200 3830 60  0001 L CNN
 F 3 "\\cern.ch\\dfs\\Applications\\Altium\\Datasheets\\R0603_NIC_NRC.pdf" H 4200 4460 60  0001 L CNN
 F 4 "100" V 4395 4910 50  0000 L CNN "~"
@@
 F 0 "R68" V 8204 5210 50  0000 L CNN
 F 1 "R0603_1K_1%_0.1W_100PPM" H 8100 4940 60  0001 L CNN
-F 2 "RESC1608X55N" H 8100 4130 60  0001 L CNN
+F 2 "Resistors SMD:RESC1608X55N" H 8100 4130 60  0001 L CNN
 F 3 "\\cern.ch\\dfs\\Applications\\Altium\\Datasheets\\R0603_NIC_NRC.pdf" H 8100 4760 60  0001 L CNN
 F 4 "1k" V 8295 5210 50  0000 L CNN "~"
@@
 F 0 "R69" V 8204 5710 50  0000 L CNN
 F 1 "R0603_1K_1%_0.1W_100PPM" H 8100 5440 60  0001 L CNN
-F 2 "RESC1608X55N" H 8100 4630 60  0001 L CNN
+F 2 "Resistors SMD:RESC1608X55N" H 8100 4630 60  0001 L CNN
 F 3 "\\cern.ch\\dfs\\Applications\\Altium\\Datasheets\\R0603_NIC_NRC.pdf" H 8100 5260 60  0001 L CNN
 F 4 "1k" V 8295 5710 50  0000 L CNN "~"
@@
 F 0 "C65" V 8504 5260 50  0000 L CNN
 F 1 "CC0603_100NF_100V_10%_X7R" H 8400 4890 60  0001 L CNN
-F 2 "CAPC1608X90N" H 8400 4080 60  0001 L CNN
+F 2 "Capacitors SMD:CAPC1608X90N" H 8400 4080 60  0001 L CNN
 F 3 "\\cern.ch\\dfs\\Applications\\Altium\\Datasheets\\CC0603_MURATA_GRM188R72A104KA35D.pdf" H 8400 4710 60  0001 L CNN
 F 4 "100nF" V 8595 5260 50  0000 L CNN "~"
@@
 F 0 "C71" V 8504 5760 50  0000 L CNN
 F 1 "CC0603_100NF_100V_10%_X7R" H 8400 5390 60  0001 L CNN
-F 2 "CAPC1608X90N" H 8400 4580 60  0001 L CNN
+F 2 "Capacitors SMD:CAPC1608X90N" H 8400 4580 60  0001 L CNN
 F 3 "\\cern.ch\\dfs\\Applications\\Altium\\Datasheets\\CC0603_MURATA_GRM188R72A104KA35D.pdf" H 8400 5210 60  0001 L CNN
 F 4 "100nF" V 8595 5760 50  0000 L CNN "~"
@@
 F 0 "C64" V 3304 6210 50  0000 L CNN
 F 1 "CC0603_1UF_50V_10%_X5R" H 3200 5840 60  0001 L CNN
-F 2 "CAPC1608X87N" H 3200 5030 60  0001 L CNN
+F 2 "Capacitors SMD:CAPC1608X87N" H 3200 5030 60  0001 L CNN
 F 3 "\\cern.ch\\dfs\\Applications\\Altium\\Datasheets\\CC0603_X5R_TDK_C.pdf" H 3200 5660 60  0001 L CNN
 F 4 "1uF" V 3395 6210 50  0000 L CNN "~"
@@
 F 0 "C67" V 3654 6210 50  0000 L CNN
 F 1 "CC0603_100NF_100V_10%_X7R" H 3550 5840 60  0001 L CNN
-F 2 "CAPC1608X90N" H 3550 5030 60  0001 L CNN
+F 2 "Capacitors SMD:CAPC1608X90N" H 3550 5030 60  0001 L CNN
 F 3 "\\cern.ch\\dfs\\Applications\\Altium\\Datasheets\\CC0603_MURATA_GRM188R72A104KA35D.pdf" H 3550 5660 60  0001 L CNN
 F 4 "100nF" V 3745 6210 50  0000 L CNN "~"
@@
 F 0 "C75" V 4054 6210 50  0000 L CNN
 F 1 "CC0603_100NF_100V_10%_X7R" H 3950 5840 60  0001 L CNN
-F 2 "CAPC1608X90N" H 3950 5030 60  0001 L CNN
+F 2 "Capacitors SMD:CAPC1608X90N" H 3950 5030 60  0001 L CNN
 F 3 "\\cern.ch\\dfs\\Applications\\Altium\\Datasheets\\CC0603_MURATA_GRM188R72A104KA35D.pdf" H 3950 5660 60  0001 L CNN
 F 4 "100nF" V 4145 6210 50  0000 L CNN "~"
@@
 F 0 "C72" V 4404 6210 50  0000 L CNN
 F 1 "CC0603_100NF_100V_10%_X7R" H 4300 5840 60  0001 L CNN
-F 2 "CAPC1608X90N" H 4300 5030 60  0001 L CNN
+F 2 "Capacitors SMD:CAPC1608X90N" H 4300 5030 60  0001 L CNN
 F 3 "\\cern.ch\\dfs\\Applications\\Altium\\Datasheets\\CC0603_MURATA_GRM188R72A104KA35D.pdf" H 4300 5660 60  0001 L CNN
 F 4 "100nF" V 4495 6210 50  0000 L CNN "~"
@@
 F 0 "C73" V 4754 6210 50  0000 L CNN
 F 1 "CC0603_100NF_100V_10%_X7R" H 4650 5840 60  0001 L CNN
-F 2 "CAPC1608X90N" H 4650 5030 60  0001 L CNN
+F 2 "Capacitors SMD:CAPC1608X90N" H 4650 5030 60  0001 L CNN
 F 3 "\\cern.ch\\dfs\\Applications\\Altium\\Datasheets\\CC0603_MURATA_GRM188R72A104KA35D.pdf" H 4650 5660 60  0001 L CNN
 F 4 "100nF" V 4845 6210 50  0000 L CNN "~"
@@
 F 0 "C11" V 5104 6210 50  0000 L CNN
 F 1 "CC0603_100NF_100V_10%_X7R" H 5000 5840 60  0001 L CNN
-F 2 "CAPC1608X90N" H 5000 5030 60  0001 L CNN
+F 2 "Capacitors SMD:CAPC1608X90N" H 5000 5030 60  0001 L CNN
 F 3 "\\cern.ch\\dfs\\Applications\\Altium\\Datasheets\\CC0603_MURATA_GRM188R72A104KA35D.pdf" H 5000 5660 60  0001 L CNN
 F 4 "100nF" V 5195 6210 50  0000 L CNN "~"
@@
 F 0 "C68" V 5454 6210 50  0000 L CNN
 F 1 "CC0603_10NF_50V_10%_X7R" H 5350 5840 60  0001 L CNN
-F 2 "CAPC1608X87N" H 5350 5030 60  0001 L CNN
+F 2 "Capacitors SMD:CAPC1608X87N" H 5350 5030 60  0001 L CNN
 F 3 "\\cern.ch\\dfs\\Applications\\Altium\\Datasheets\\CC0603_X7R_PHYCOMP.pdf" H 5350 5660 60  0001 L CNN
 F 4 "10nF" V 5545 6210 50  0000 L CNN "~"
@@
 F 0 "C69" V 5804 6210 50  0000 L CNN
 F 1 "CC0603_10NF_50V_10%_X7R" H 5700 5840 60  0001 L CNN
-F 2 "CAPC1608X87N" H 5700 5030 60  0001 L CNN
+F 2 "Capacitors SMD:CAPC1608X87N" H 5700 5030 60  0001 L CNN
 F 3 "\\cern.ch\\dfs\\Applications\\Altium\\Datasheets\\CC0603_X7R_PHYCOMP.pdf" H 5700 5660 60  0001 L CNN
 F 4 "10nF" V 5895 6210 50  0000 L CNN "~"
@@
 F 0 "C70" V 6154 6210 50  0000 L CNN
 F 1 "CC0603_10NF_50V_10%_X7R" H 6050 5840 60  0001 L CNN
-F 2 "CAPC1608X87N" H 6050 5030 60  0001 L CNN
+F 2 "Capacitors SMD:CAPC1608X87N" H 6050 5030 60  0001 L CNN
 F 3 "\\cern.ch\\dfs\\Applications\\Altium\\Datasheets\\CC0603_X7R_PHYCOMP.pdf" H 6050 5660 60  0001 L CNN
 F 4 "10nF" V 6245 6210 50  0000 L CNN "~"
@@
 F 0 "C66" V 6504 6210 50  0000 L CNN
 F 1 "CC0603_10NF_50V_10%_X7R" H 6400 5840 60  0001 L CNN
-F 2 "CAPC1608X87N" H 6400 5030 60  0001 L CNN
+F 2 "Capacitors SMD:CAPC1608X87N" H 6400 5030 60  0001 L CNN
 F 3 "\\cern.ch\\dfs\\Applications\\Altium\\Datasheets\\CC0603_X7R_PHYCOMP.pdf" H 6400 5660 60  0001 L CNN
 F 4 "10nF" V 6595 6210 50  0000 L CNN "~"

Commit message: Completed port to KiCad, passes DRC+LVS. NOT MANUFACTURED.
Parts:
- IC10: footprint (none) -> dsi_shield:TSOP66
Changed lines of the file:
@@
 F 0 "IC10" H 4500 7425 50  0000 C CNN
 F 1 "MT46V32M16P-5B:F" H 4875 7325 60  0000 C CNN
-F 2 "" H 7650 3400 60  0001 L CNN
+F 2 "dsi_shield:TSOP66" H 7650 3400 60  0001 L CNN
 F 3 "" H 7650 3310 60  0001 L CNN
 F 4 "Value" H 7650 4450 60  0001 C CNN "Fieldname"

Commit message: axi4/zynq version: wip
Parts:
- C11, C65, C67, C71, C72, C73, C75: symbol CC0603_100NF_100V_10%_X7R -> dsi_shield-rescue:CC0603_100NF_100V_10%_X7R-
- C64: symbol CC0603_1UF_50V_10%_X5R -> dsi_shield-rescue:CC0603_1UF_50V_10%_X5R-
- C66, C68, C69, C70: symbol CC0603_10NF_50V_10%_X7R -> dsi_shield-rescue:CC0603_10NF_50V_10%_X7R-
- IC10: symbol MT46V32M16P-5B:F -> dsi_shield-rescue:F-MT46V32M16P-5B
- R67: symbol R0603_100R_1%_0.1W_100PPM -> dsi_shield-rescue:R0603_100R_1%_0.1W_100PPM-
- R68, R69: symbol R0603_1K_1%_0.1W_100PPM -> dsi_shield-rescue:R0603_1K_1%_0.1W_100PPM-
Changed lines of the file:
@@
-EESchema Schematic File Version 2
-LIBS:Capacitors Networks THD
-LIBS:Capacitors Networks SMD
-LIBS:Capacitors THD
-LIBS:Capacitors SMD
-LIBS:Miscellaneous
-LIBS:HARWIN
-LIBS:LEMO
-LIBS:WEIDMULLER
-LIBS:FCI
-LIBS:MOLEX
-LIBS:TYCO
-LIBS:ERNI
-LIBS:MENTOR
-LIBS:SAMTEC
-LIBS:STELVIO-KONTEK COMATEL
-LIBS:AMPHENOL
-LIBS:HARTING
-LIBS:3M
-LIBS:Pads
-LIBS:Switches
-LIBS:Relays
-LIBS:Heat-Sinks
-LIBS:Fasteners & Fixings
-LIBS:Batteries
-LIBS:Fuses
-LIBS:Metal Screening Box
-LIBS:Sockets
-LIBS:Regulators
-LIBS:Transistors
-LIBS:Power Supplies
-LIBS:Analog & Interface
-LIBS:Sensors
-LIBS:Logic
-LIBS:Optocouplers
-LIBS:Standard Logic
-LIBS:DC-DC Converters
-LIBS:Operational Amplifiers
-LIBS:Crystals & Oscillators
-LIBS:Diodes
-LIBS:LEDs & Displays
-LIBS:PCB Modules
-LIBS:Bonding
-LIBS:Resistors THD
-LIBS:Potentiometers SMD
-LIBS:Thermistors And Varistors
-LIBS:Potentiometers THD
-LIBS:Resistor Networks THD
-LIBS:Resistors SMD
-LIBS:Resistor Networks SMD
-LIBS:Transformers
-LIBS:Inductors SMD
-LIBS:Inductors THD
-LIBS:Cores
-LIBS:power
-LIBS:conn
-LIBS:dsi_shield
+EESchema Schematic File Version 4
 LIBS:dsi_shield-cache
 EELAYER 26 0
@@
 $EndDescr
 $Comp
-L MT46V32M16P-5B:F IC10
+L dsi_shield-rescue:F-MT46V32M16P-5B IC10
 U 1 1 59956E83
 P 7650 4450
@@
 $EndComp
 $Comp
-L +2V5 #PWR093
+L dsi_shield-rescue:+2V5- #PWR093
 U 1 1 59957939
 P 5450 1050
@@
 SDRAM_CLK_N
 $Comp
-L R0603_100R_1%_0.1W_100PPM R67
+L dsi_shield-rescue:R0603_100R_1%_0.1W_100PPM- R67
 U 1 1 5995CCB9
 P 4200 4850
@@
 Connection ~ 5450 5350
 $Comp
-L GND #PWR094
+L dsi_shield-rescue:GND- #PWR094
 U 1 1 5995E2A8
 P 5450 5500
@@
 	7800 5550 8400 5550
 $Comp
-L R0603_1K_1%_0.1W_100PPM R68
+L dsi_shield-rescue:R0603_1K_1%_0.1W_100PPM- R68
 U 1 1 599686D8
 P 8100 5150
@@
 $EndComp
 $Comp
-L R0603_1K_1%_0.1W_100PPM R69
+L dsi_shield-rescue:R0603_1K_1%_0.1W_100PPM- R69
 U 1 1 59968851
 P 8100 5650
@@
 $EndComp
 $Comp
-L CC0603_100NF_100V_10%_X7R C65
+L dsi_shield-rescue:CC0603_100NF_100V_10%_X7R- C65
 U 1 1 5996A953
 P 8400 5150
@@
 $EndComp
 $Comp
-L CC0603_100NF_100V_10%_X7R C71
+L dsi_shield-rescue:CC0603_100NF_100V_10%_X7R- C71
 U 1 1 5996AB59
 P 8400 5650
@@
 Connection ~ 8100 5050
 $Comp
-L +2V5 #PWR095
+L dsi_shield-rescue:+2V5- #PWR095
 U 1 1 5996C81F
 P 8100 4950
@@
 Connection ~ 8100 6050
 $Comp
-L GND #PWR096
+L dsi_shield-rescue:GND- #PWR096
 U 1 1 5996C96D
 P 8100 6150
@@
 DDR SDRAM
 $Comp
-L CC0603_1UF_50V_10%_X5R C64
+L dsi_shield-rescue:CC0603_1UF_50V_10%_X5R- C64
 U 1 1 59971751
 P 3200 6100
@@
 $EndComp
 $Comp
-L CC0603_100NF_100V_10%_X7R C67
+L dsi_shield-rescue:CC0603_100NF_100V_10%_X7R- C67
 U 1 1 599729A9
 P 3550 6100
@@
 $EndComp
 $Comp
-L CC0603_100NF_100V_10%_X7R C75
+L dsi_shield-rescue:CC0603_100NF_100V_10%_X7R- C75
 U 1 1 59972AF3
 P 3950 6100
@@
 $EndComp
 $Comp
-L CC0603_100NF_100V_10%_X7R C72
+L dsi_shield-rescue:CC0603_100NF_100V_10%_X7R- C72
 U 1 1 59972B6B
 P 4300 6100
@@
 $EndComp
 $Comp
-L CC0603_100NF_100V_10%_X7R C73
+L dsi_shield-rescue:CC0603_100NF_100V_10%_X7R- C73
 U 1 1 59972BE5
 P 4650 6100
@@
 $EndComp
 $Comp
-L CC0603_100NF_100V_10%_X7R C11
+L dsi_shield-rescue:CC0603_100NF_100V_10%_X7R- C11
 U 1 1 59972C5F
 P 5000 6100
@@
 $EndComp
 $Comp
-L CC0603_10NF_50V_10%_X7R C68
+L dsi_shield-rescue:CC0603_10NF_50V_10%_X7R- C68
 U 1 1 5997381F
 P 5350 6100
@@
 $EndComp
 $Comp
-L CC0603_10NF_50V_10%_X7R C69
+L dsi_shield-rescue:CC0603_10NF_50V_10%_X7R- C69
 U 1 1 59973B76
 P 5700 6100
@@
 $EndComp
 $Comp
-L CC0603_10NF_50V_10%_X7R C70
+L dsi_shield-rescue:CC0603_10NF_50V_10%_X7R- C70
 U 1 1 59973BF6
 P 6050 6100
@@
 $EndComp
 $Comp
-L CC0603_10NF_50V_10%_X7R C66
+L dsi_shield-rescue:CC0603_10NF_50V_10%_X7R- C66
 U 1 1 59973C78
 P 6400 6100
@@
 Connection ~ 6050 6500
 $Comp
-L +2V5 #PWR097
+L dsi_shield-rescue:+2V5- #PWR097
 U 1 1 5997637D
 P 3200 5900
@@
 Connection ~ 3200 6000
 $Comp
-L GND #PWR098
+L dsi_shield-rescue:GND- #PWR098
 U 1 1 59976555
 P 3200 6600
